File: pcb/lineSensor.kicad_pcb (KiCad board)
At the start: 2 copper layers, 82 x 22.7 mm, 32 parts, among them J1 Conn_01x07, Q1 BC817, U1 ITR8307, U2 ITR8307, U3 ITR8307, U4 ITR8307, U5 ITR8307, U6 ITR8307, U7 ITR8307, U8 ITR8307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

Commit message: PCB: improve line sensor board
- change size of SMD parts from 0603 to 1206
- change name of board from SensorLine to RB0001-LineSensor
- change version v0.2 to v0.3
- add license CC BY-SA 4.0
- add information about repository github:roboticsbrno/RB0001-LineSensor
Parts:
- C1: footprint Capacitor_SMD:C_0603_1608Metric_Pad1.05x0.95mm_HandSolder -> Capacitor_SMD:C_1206_3216Metric_Pad1.42x1.75mm_HandSolder
- J1: moved to B.Cu
- R1, R10, R11, R12, R13, R14, R15, R16, R17, R2, R3, R4, R5, R6, R7, R8, R9: footprint Resistor_SMD:R_0603_1608Metric_Pad1.05x0.95mm_HandSolder -> Resistor_SMD:R_1206_3216Metric_Pad1.42x1.75mm_HandSolder
- moved R1 0.56 mm to (178.4, 105.1)
- moved R4 0.49 mm to (151.5, 98.0)
- moved R3 0.49 mm to (159.5, 99.1)
- moved R8 0.48 mm to (118.6, 105.1)
- moved R2 0.47 mm to (168.5, 101.1)
- moved R6 0.46 mm to (137.5, 99.1)
- moved R5 0.46 mm to (145.5, 97.9)
- moved R7 0.35 mm to (128.7, 100.9)
- turned J1 to 90 degrees
Other:
- board text added: "RB0001-LineSensor v0.3 06/2019 CC BY-SA 4.0"
- board text added: "github:roboticsbrno/RB0001-LineSensor"
- board text removed: "SensorLine v0.2 11/2018"

Commit message: PCB: add signalization LEDs, copy pins labels (F.SilkS => B.SilkS)
- add power and back-light signalization LEDs
Parts:
- added D1: LED_GREEN, LED_SMD:LED_1206_3216Metric_Pad1.42x1.75mm_HandSolder, B.Cu at (147.3, 106.8)
- added D2: LED_RED, LED_SMD:LED_1206_3216Metric_Pad1.42x1.75mm_HandSolder, B.Cu at (132.5, 111.0)
- added R18: 220R, Resistor_SMD:R_1206_3216Metric_Pad1.42x1.75mm_HandSolder, B.Cu at (147.3, 110.5)
- added R19: 220R, Resistor_SMD:R_1206_3216Metric_Pad1.42x1.75mm_HandSolder, B.Cu at (126.3, 111.0)
Routing:
- net GND: track 14.3 -> 18.7 mm
- net LED_GND: track 81.6 -> 84.9 mm
- net Net-(D1-Pad2): track 0.00 -> 3.30 mm
- net Net-(D2-Pad2): track 0.00 -> 3.18 mm
Other:
- board text added: "GND VDD SCK MISO MOSI CS LED"
